File: packages/ebyte-e73/layouts/usage/usage.kicad_pcb (KiCad board)
At the start: 2 copper layers, 3 parts

Commit message: adding has_part_picked trait to all
Parts:
- added R1: 10kΩ ±1% 62.5mW, UNI_ROYAL_0402WGF1002TCE:R0402, F.Cu at (0.00, 0.00)
- moved C1 10.0 mm to (10.0, -10.0)
- moved C2 10.0 mm to (10.0, -20.0)
- moved U1 10.0 mm to (10.0, 0.00)
Connections:
- net P0_03 renamed gpio[2]-line
- net P1_10 renamed gpio[1]-line
- net P1_11 renamed gpio[0]-line
