File: packages/ti-bq25798/layouts/default/default.kicad_pcb (KiCad board)
At the start: 2 copper layers, 7 parts

Commit message: BQ25798
Parts:
- added R1: 390Ω ±1% 100mW, PANASONIC_ERJ2RKF3900X:R0402, F.Cu at (0.00, 0.00)
